File: Hardware/01_Design/02_KiCad/IgnitionController/IgnitionDriver.kicad_sch (KiCad schematic)
At the start: 0 parts

Commit message: Peripherals Update
Parts:
- added D17, D18, D6, D7: SM6T100A, Diode_SMD:D_SMB, symbol Diode:SM6T100A
- added Q10, Q11, Q8, Q9: IRF540N, Package_TO_SOT_THT:TO-220-3_Vertical, symbol Transistor_FET:IRF540N
- added R54, R55, R56, R61: 100R, symbol Device:R_Small
Connections:
- new net: Q11.1 (G), R56.2
- new net: Q8.1 (G), R61.2
- new net: Q10.1 (G), R54.2
- new net: Q9.1 (G), R55.2
- new net GND: D17.2 (A2), D18.2 (A2), D6.2 (A2), D7.2 (A2), Q10.3 (S), Q11.3 (S), Q8.3 (S), Q9.3 (S)
- new net IGN_COIL_1: D6.1 (A1), Q8.2 (D)
- new net IGN_COIL_2: D7.1 (A1), Q9.2 (D)
- new net IGN_COIL_3: D17.1 (A1), Q10.2 (D)
- new net IGN_COIL_4: D18.1 (A1), Q11.2 (D)
- new net IGN_COIL_DRV_1: R61.1
- new net IGN_COIL_DRV_2: R55.1
- new net IGN_COIL_DRV_3: R54.1
- new net IGN_COIL_DRV_4: R56.1

Commit message: Updates to HW Layout
Parts:
- R54, R55, R56, R61: footprint (none) -> Resistor_SMD:R_0805_2012Metric_Pad1.20x1.40mm_HandSolder
Changed lines of the file:
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@@
 			)
 		)
-		(property "Footprint" ""
+		(property "Footprint" "Resistor_SMD:R_0805_2012Metric_Pad1.20x1.40mm_HandSolder"
 			(at 53.34 113.03 0)
 			(effects
@@
 			)
 		)
-		(property "Footprint" ""
+		(property "Footprint" "Resistor_SMD:R_0805_2012Metric_Pad1.20x1.40mm_HandSolder"
 			(at 53.34 86.36 0)
 			(effects
@@
 			)
 		)
-		(property "Footprint" ""
+		(property "Footprint" "Resistor_SMD:R_0805_2012Metric_Pad1.20x1.40mm_HandSolder"
 			(at 53.34 62.23 0)
 			(effects
@@
 			)
 		)
-		(property "Footprint" ""
+		(property "Footprint" "Resistor_SMD:R_0805_2012Metric_Pad1.20x1.40mm_HandSolder"
 			(at 53.34 36.83 0)
 			(effects

Commit message: Initial routing of Power supply
Parts:
- R54, R55, R56, R61: footprint Resistor_SMD:R_0805_2012Metric_Pad1.20x1.40mm_HandSolder -> Resistor_SMD:R_0603_1608Metric_Pad0.98x0.95mm_HandSolder
Changed lines of the file:
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@@
 			)
 		)
-		(property "Footprint" "Resistor_SMD:R_0805_2012Metric_Pad1.20x1.40mm_HandSolder"
+		(property "Footprint" "Resistor_SMD:R_0603_1608Metric_Pad0.98x0.95mm_HandSolder"
 			(at 53.34 113.03 0)
 			(effects
@@
 			)
 		)
-		(property "Footprint" "Resistor_SMD:R_0805_2012Metric_Pad1.20x1.40mm_HandSolder"
+		(property "Footprint" "Resistor_SMD:R_0603_1608Metric_Pad0.98x0.95mm_HandSolder"
 			(at 53.34 86.36 0)
 			(effects
@@
 			)
 		)
-		(property "Footprint" "Resistor_SMD:R_0805_2012Metric_Pad1.20x1.40mm_HandSolder"
+		(property "Footprint" "Resistor_SMD:R_0603_1608Metric_Pad0.98x0.95mm_HandSolder"
 			(at 53.34 62.23 0)
 			(effects
@@
 			)
 		)
-		(property "Footprint" "Resistor_SMD:R_0805_2012Metric_Pad1.20x1.40mm_HandSolder"
+		(property "Footprint" "Resistor_SMD:R_0603_1608Metric_Pad0.98x0.95mm_HandSolder"
 			(at 53.34 36.83 0)
 			(effects
